File: Proyecto final/Kicad/tps63020/tps63020.kicad_pcb (KiCad board)
At the start: 4 copper layers, 23 parts, among them U2 TPS63020DSJR

Commit message: Enrutado TPS63020
Routing:
- net Net-(U2-FB): track 16.7 -> 17.7 mm
- removed copper zone on In2.Cu, net VBAT
Changed lines of the file:
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@@
 		(capping no)
 		(filling no)
-		(zone_defaults)
 		(pcbplotparams
 			(layerselection 0x00000000_00000000_55555555_5755f5ff)
@@
 		(at 135.2 60 180)
 		(property "Reference" "U2"
-			(at 25.357979 13 0)
+			(at -0.05 13 0)
 			(layer "F.SilkS")
 			(effects
@@
 		)
 	)
+	(segment
+		(start 128.5375 59.8375)
+		(end 126.675 59.8375)
+		(width 0.25)
+		(layer "F.Cu")
+		(net "VBAT")
+	)
+	(segment
+		(start 131.8 63.1)
+		(end 128.5375 59.8375)
+		(width 0.25)
+		(layer "F.Cu")
+		(net "VBAT")
+	)
+	(segment
+		(start 136.575 61.5)
+		(end 136.575 61.675)
+		(width 0.25)
+		(layer "F.Cu")
+		(net "VBAT")
+	)
+	(segment
+		(start 136.575 61.675)
+		(end 137.1 62.2)
+		(width 0.25)
+		(layer "F.Cu")
+		(net "VBAT")
+	)
+	(segment
+		(start 136.6 61.525)
+		(end 136.575 61.5)
+		(width 0.25)
+		(layer "F.Cu")
+		(net "VBAT")
+	)
 	(via
-		(at 144.2 63)
+		(at 131.8 63.1)
+		(size 0.6)
+		(drill 0.3)
+		(layers "F.Cu" "B.Cu")
+		(net "VBAT")
+	)
+	(via
+		(at 126.3 61.7)
 		(size 0.6)
 		(drill 0.3)
 		(layers "F.Cu" "B.Cu")
 		(free yes)
-		(net "+3V3")
+		(net "VBAT")
+	)
+	(via
+		(at 137.1 62.2)
+		(size 0.6)
+		(drill 0.3)
+		(layers "F.Cu" "B.Cu")
+		(net "VBAT")
+	)
+	(segment
+		(start 133.5 64.8)
+		(end 131.8 63.1)
+		(width 0.25)
+		(layer "In2.Cu")
+		(net "VBAT")
+	)
+	(segment
+		(start 137.1 64.4)
+		(end 136.7 64.8)
+		(width 0.25)
+		(layer "In2.Cu")
+		(net "VBAT")
+	)
+	(segment
+		(start 137.1 62.2)
+		(end 137.1 64.4)
+		(width 0.25)
+		(layer "In2.Cu")
+		(net "VBAT")
+	)
+	(segment
+		(start 136.7 64.8)
+		(end 133.5 64.8)
+		(width 0.25)
+		(layer "In2.Cu")
+		(net "VBAT")
 	)
 	(segment
@@
 	)
 	(segment
-		(start 136.909325 60.5)
-		(end 136.6 60.5)
+		(start 138.05 61.640675)
+		(end 136.909325 60.5)
 		(width 0.25)
 		(layer "F.Cu")
@@
 	)
 	(segment
-		(start 137.7 61.4)
-		(end 137.7 61.290675)
+		(start 138.05 63.45)
+		(end 138.05 61.640675)
 		(width 0.25)
 		(layer "F.Cu")
@@
 	)
 	(segment
-		(start 137.7 61.290675)
-		(end 136.909325 60.5)
+		(start 147.6 62.9)
+		(end 147.6 64.1)
 		(width 0.25)
 		(layer "F.Cu")
@@
 	)
 	(segment
-		(start 147.6 62.9)
-		(end 147.6 64.1)
+		(start 148 62.5)
+		(end 147.6 62.9)
 		(width 0.25)
 		(layer "F.Cu")
@@
 	)
 	(segment
-		(start 148 62.5)
-		(end 147.6 62.9)
+		(start 136.909325 60.5)
+		(end 136.6 60.5)
 		(width 0.25)
 		(layer "F.Cu")
@@
 	)
 	(via
-		(at 137.7 61.4)
+		(at 138.05 63.45)
 		(size 0.6)
 		(drill 0.3)
@@
 	)
 	(segment
-		(start 147.6 64.1)
-		(end 140.4 64.1)
+		(start 138.7 64.1)
+		(end 147.6 64.1)
 		(width 0.25)
 		(layer "B.Cu")
@@
 	)
 	(segment
-		(start 140.4 64.1)
-		(end 137.7 61.4)
+		(start 138.05 63.45)
+		(end 138.7 64.1)
 		(width 0.25)
 		(layer "B.Cu")
 		(net "Net-(U2-FB)")
 	)
-	(segment
-		(start 128.5375 59.8375)
-		(end 126.675 59.8375)
-		(width 0.25)
-		(layer "F.Cu")
-		(net "VBAT")
-	)
-	(segment
-		(start 131.8 63.1)
-		(end 128.5375 59.8375)
-		(width 0.25)
-		(layer "F.Cu")
-		(net "VBAT")
-	)
-	(segment
-		(start 136.575 61.5)
-		(end 136.575 61.675)
-		(width 0.25)
-		(layer "F.Cu")
-		(net "VBAT")
-	)
-	(segment
-		(start 136.575 61.675)
-		(end 137.1 62.2)
-		(width 0.25)
-		(layer "F.Cu")
-		(net "VBAT")
-	)
-	(segment
-		(start 136.6 61.525)
-		(end 136.575 61.5)
-		(width 0.25)
-		(layer "F.Cu")
-		(net "VBAT")
-	)
 	(via
-		(at 131.8 63.1)
-		(size 0.6)
-		(drill 0.3)
-		(layers "F.Cu" "B.Cu")
-		(net "VBAT")
-	)
-	(via
-		(at 126.3 61.7)
+		(at 144.2 63)
 		(size 0.6)
 		(drill 0.3)
 		(layers "F.Cu" "B.Cu")
 		(free yes)
-		(net "VBAT")
-	)
-	(via
-		(at 137.1 62.2)
-		(size 0.6)
-		(drill 0.3)
-		(layers "F.Cu" "B.Cu")
-		(net "VBAT")
-	)
-	(segment
-		(start 133.5 64.8)
-		(end 131.8 63.1)
-		(width 0.25)
-		(layer "In2.Cu")
-		(net "VBAT")
-	)
-	(segment
-		(start 137.1 64.4)
-		(end 136.7 64.8)
-		(width 0.25)
-		(layer "In2.Cu")
-		(net "VBAT")
-	)
-	(segment
-		(start 137.1 62.2)
-		(end 137.1 64.4)
-		(width 0.25)
-		(layer "In2.Cu")
-		(net "VBAT")
-	)
-	(segment
-		(start 136.7 64.8)
-		(end 133.5 64.8)
-		(width 0.25)
-		(layer "In2.Cu")
-		(net "VBAT")
+		(net "+3V3")
 	)
 	(segment
@@
 		(priority 2)
 		(connect_pads yes
-			(clearance 0.5)
+			(clearance 0.25)
 		)
 		(min_thickness 0.25)
@@
 		(priority 5)
 		(connect_pads yes
-			(clearance 0.2)
+			(clearance 0.25)
 		)
-		(min_thickness 0.2)
+		(min_thickness 0.25)
 		(fill yes
 			(thermal_gap 0.5)
@@
 		(priority 3)
 		(connect_pads yes
-			(clearance 0.5)
+			(clearance 0.25)
 		)
 		(min_thickness 0.25)
@@
 	)
 	(zone
-		(net "Net-(U2-L2_6)")
+		(net "VBAT")
 		(layer "F.Cu")
 		(hatch edge 0.5)
-		(priority 2)
+		(priority 4)
 		(connect_pads yes
 			(clearance 0.25)
@@
 		(polygon
 			(pts
-				(xy 136.175 59.2) (xy 136.975 59.2) (xy 137.175 59) (xy 137.175 57.8) (xy 139.375 56.6) (xy 139.375 50.2)
-				(xy 136.975 50.2) (xy 136.975 56.6) (xy 136.175 58.2)
+				(xy 125.475 59.4) (xy 125.475 61.8) (xy 126.175 62.5) (xy 131.475 62.5) (xy 133.275 60.7) (xy 134.075 60.7)
+				(xy 134.075 59.4)
 			)
 		)
 	)
 	(zone
-		(net "GND")
+		(net "Net-(U2-L2_6)")
 		(layer "F.Cu")
 		(hatch edge 0.5)
-		(priority 1)
+		(priority 2)
 		(connect_pads yes
 			(clearance 0.25)
@@
 		(min_thickness 0.25)
 		(fill yes
-			(thermal_gap 0.1)
+			(thermal_gap 0.5)
 			(thermal_bridge_width 0.5)
 			(island_removal_mode 1)
@@
 		(polygon
 			(pts
-				(xy 134.375 58.2) (xy 134.375 57.6) (xy 133.675 56.912446) (xy 133.675 55.787123) (xy 136.675 55.8125)
-				(xy 136.675 56.8875) (xy 135.975 57.6) (xy 135.975 58.2)
+				(xy 136.175 59.2) (xy 136.975 59.2) (xy 137.175 59) (xy 137.175 57.8) (xy 139.375 56.6) (xy 139.375 50.2)
+				(xy 136.975 50.2) (xy 136.975 56.6) (xy 136.175 58.2)
 			)
 		)
 	)
 	(zone
-		(net "VBAT")
-		(layers "F.Cu" "In2.Cu")
+		(net "GND")
+		(layer "F.Cu")
 		(hatch edge 0.5)
-		(priority 4)
+		(priority 1)
 		(connect_pads yes
-			(clearance 0.5)
+			(clearance 0.25)
 		)
 		(min_thickness 0.25)
 		(fill yes
-			(thermal_gap 0.5)
+			(thermal_gap 0.1)
 			(thermal_bridge_width 0.5)
 			(island_removal_mode 1)
@@
 		(polygon
 			(pts
-				(xy 125.475 59.4) (xy 125.475 61.8) (xy 126.175 62.5) (xy 131.475 62.5) (xy 133.275 60.7) (xy 134.075 60.7)
-				(xy 134.075 59.4)
+				(xy 134.375 58.2) (xy 134.375 57.6) (xy 133.675 56.9) (xy 133.675 55.75) (xy 136.675 55.75) (xy 136.675 56.9)
+				(xy 135.975 57.6) (xy 135.975 58.2)
 			)
 		)
 	)
+	(group "tps63020"
+		(lib_id "TPS63020 block:tps63020")
+		(members "0013b714-ebf6-4c26-8eea-e1347709b81b" "004b255b-035a-44c0-b984-07962810cfc0"
+			"0359a73c-714a-49b5-98e4-a9ea71cff2b8" "04f34494-e531-4fe9-94a1-7e950bf645a1"
+			"074b7bcb-85f0-4d32-a9ab-f3fbe7b2b5fd" "082c52ce-7b6a-450f-ab86-be167e27ecdc"
+			"09394d96-30c4-4e07-b202-a4ee724fcfea" "0a84fe92-59a8-4ada-8f57-b8abbde472ec"
+			"0bd9cd30-57f5-4609-9517-9a82efa4bacb" "0db402c5-fd70-4adb-9d23-587764cabe45"
+			"0ebbf341-ab83-4028-a9c8-92716383e7dc" "13194350-0384-4ffd-975f-74b0493eefdb"
+			"14a51445-2586-4d3d-95a8-121a7ad4844d" "188c3e4e-547c-4f3f-8c90-03e8f99baf3c"
+			"1a4e88f7-33ac-4c06-ac8f-530e781ff730" "1d5dc650-3fd5-4768-a47c-23b0bad8fb6b"
+			"229a2e71-78d5-4627-a86f-6f8ce33d81d4" "2ce6cfe5-3ded-4044-b68a-4c4ae40b57b2"
+			"2f03fc14-33a8-4863-8662-bec5e9233dc3" "2f6ac57b-c545-4be2-9483-3f1fcbed7acd"
+			"32a3861f-5426-4867-b897-56b400cacaa5" "330b806f-9775-481c-98ac-b89c1a18879b"
+			"34ea6aad-1e4c-46e6-a880-dda1a61ce769" "38628fab-9de8-4dcd-8461-2cb59240a9c3"
+			"40c7742c-a5be-424b-87ec-bb5201782c00" "421b42ba-b339-4476-81eb-7c6eb38c1752"
+			"45114706-ae1b-4588-a9c5-27529b0f85c6" "46aabbab-ac10-432e-922d-1089492e49cf"
+			"48354d34-5c24-4e87-bcbe-aa4ec5cbe4e9" "4de9fb1c-15a9-4794-b82d-42bf42f3dfc7"
+			"4ee15b6b-5ba5-4062-a921-df61a0ce0fbc" "50e919e8-d7b3-4da6-998f-a62a7dbdaf89"
+			"52e54b3d-9b02-47b2-aabf-2b493660cd59" "5a76240f-d363-4605-9f8b-d05eab3a7221"
+			"5fd810e1-d9fc-4260-a254-5db2a9cf163f" "611bbb83-53e5-420d-a54e-e4259eb9d674"
+			"6a7bf559-c22c-4b05-ba6b-7c89e5752cdc" "6be31813-8f13-4143-be4e-08eb965f4506"
+			"6d7a50d3-5a35-4e4f-9cfd-fa8403ae2618" "6e80771d-39f7-42b0-9340-3f3a51b2c9c9"
+			"70f07e38-ba0c-476a-8171-4bb464c2f04a" "735700cd-5de3-429f-93b9-83478aae55ae"
+			"7bf01175-1aa5-4c9d-b4fc-44744bcd5ca9" "7c2151f8-b0f9-4046-896a-15bce030e001"
+			"7d626905-2d5a-4759-9025-6ce912813119" "801123d0-60d6-45db-9b19-77e9b03e6920"
+			"8356b9ae-469a-4983-a679-883ebcdcc42b" "879fe100-0263-4276-85c5-0c592a614177"
+			"8af008ac-109f-4be2-938c-0330bc324a3c" "8df789f2-9650-4a76-ae61-6a2709b8ac1f"
+			"93bd9dc1-460d-4479-a1ae-ad790fb0af19" "97a1b1d7-ee80-4628-9070-8dbb539ce46f"
+			"9a52bebf-5d54-47f9-88c0-64e020c146b7" "9c7aa14d-5c8f-40ec-8b75-d44e50c9ef73"
+			"9d4d5c08-6e42-4ed2-801e-ee16b41fe1c2" "a0d7d095-139a-469a-8629-14a98bcc6178"
+			"a6d890f4-1325-45b3-8b6d-d654a84836c5" "aa50cfda-ea58-4932-a3ba-2121249f14d2"
+			"aa98ded6-d4c4-4d59-842a-b1992c02b8ad" "acb5aae7-6150-4f59-8dfe-f769941a64c9"
+			"aefb934d-fe28-4cf5-a93c-4ae6247237e2" "b016ad98-20fe-43e9-9111-a60f9cb5abe3"
+			"b3f176c7-a7d9-43ab-a28b-6a5ffa451533" "c094726e-68e1-4b53-90cf-863806d03f39"
+			"c1ee7433-bed6-4bb4-804a-0f0e0fef9cf5" "c3a2f53c-8f1a-4331-80c8-396498cb7302"
+			"c52520ac-ada5-4145-b521-abca01f5ada4" "d0f1e173-c428-4e21-990d-9eeee1113b3d"
+			"dc24b931-0983-4ac5-8b30-6b7946000b37" "df886b06-d3f4-4a3e-b012-d586143bb6a4"
+			"e11578ac-ddb1-428a-9dc7-97f90a2c598e" "e17abc7b-c0ae-4df9-974c-3a1961efb867"
+			"e2749f09-d77a-42da-bf8a-be52d8e29f7b" "e4bb4a2f-5668-4021-a319-690f82334b88"
+			"e6b911a7-fc92-415f-bdb4-d68d4dc92dfa" "e9d27ca0-6be9-47b3-90a5-82a4756f3d18"
+			"eb748d87-2c6b-4f0e-8128-324d789defbf" "effc1e88-bfae-4c03-a99c-5f74c4717589"
+			"f2debaa3-9310-413a-9ffc-6b08ac9cd9b4" "f63596f4-9867-46a5-9b08-4e46a9c1214d"
+			"f6fbeccc-68f0-4bd5-9572-9df6ac55da85" "f8da0680-5001-4784-968e-c6d6be956d5e"
+			"fb08bee7-0e92-4564-850e-a695c5976ee5" "fb38e04d-d98e-4ab7-8d04-54010047a1a4"
+			"fbd13940-9133-4cff-8234-874018cc23eb" "fd6a7108-195b-4184-9c43-da2aaa5d4046"
+		)
+	)
