File: Proyecto final/Kicad/Guantes traductores/Guantes traductores.kicad_pcb (KiCad board)
At the start: 4 copper layers, 66.7 x 54.2 mm, 96 parts, among them J1 USB_C_Receptacle_USB2.0_16P, J10 Contacto1, J11 Contacto2, J12 Contacto3, J13 Contacto4, J3 Flex1, J4 Flex2, J5 Flex3, J6 Flex4, J7 Flex5, SW1 SW_SPST, SW2 SW_SPST, U1 ESP32-C3-WROOM-02, U10 TPS63020DSJR, U2 ADS7128IRTER, U3 USBLC6-2SC6, U4 LMV324, U5 LMV324, U7 TP4056 Board, U8 BNO055

Commit message: Switch y leds
Parts:
- added R28: 200, Resistor_SMD:R_0805_2012Metric, F.Cu at (144.5, 161.5)
- added R29: 200, Resistor_SMD:R_0805_2012Metric, F.Cu at (148.4, 161.5)
- added U6: SS12D10G5, lcsc_footprints:C7431054_SW-TH_SHOU-HAN_SS12D10G4, F.Cu at (133.4, 169.2)
- added U9: HSMF-C113_C6795902, lcsc_footprints:C6795902_LED-SMD_HSMF-C113, F.Cu at (146.4, 159.1)
- moved D2 14.8 mm to (146.7, 179.2), turned to 0 degrees
- moved D3 2.25 mm to (135.7, 178.0), turned to -90 degrees
- moved U7 2.25 mm to (155.5, 178.2)
Connections:
- D2 pad 1: /Buckboost 3.7V-5V a 3.3V/Vin -> Net-(D2-K)
- D3 pad 1: /Buckboost 3.7V-5V a 3.3V/Vin -> Net-(D2-K)
Routing:
- net IO10: track 0.00 -> 12.3 mm
- net GND: track 85.6 -> 94.5 mm
- net Net-(R28-Pad2): track 0.00 -> 2.79 mm
- net Net-(R29-Pad2): track 0.00 -> 2.67 mm
- net +3.3V: track 83.5 -> 85.6 mm, vias 24 -> 25
- net VBat: track 29.7 -> 30.6 mm
- added copper zone on F.Cu, net Net-(D2-K)

Commit message: Ajustes y mounting holes
Parts:
- added H1: MountingHole_2.2mm_M2_ISO7380_Pad_TopOnly, MountingHole:MountingHole_2.2mm_M2_ISO7380_Pad_TopOnly, F.Cu at (154.9, 138.3)
- added H2: MountingHole_2.2mm_M2_ISO7380_Pad_TopOnly, MountingHole:MountingHole_2.2mm_M2_ISO7380_Pad_TopOnly, F.Cu at (119.5, 180.0)
Routing:
- net +3.3V: track 85.6 -> 57.0 mm
Other:
- board size 66.7 x 54.2 mm -> 66.5 x 55.5 mm

Commit message: Preparacion para pedido JLCPCB
Parts:
- D2, D3: value PMEG6010CEH -> SMD26PL-TP
- R14, R15, R16, R22, R24: value 100k -> 250k
- moved U9 0.05 mm to (146.4, 159.1)
Other:
- board text added: "PF_LSD_G3_J"

Commit message: Ajustes vias de esp32
Parts:
- added J2: Conn_01x03_Pin, Connector_PinHeader_2.54mm:PinHeader_1x03_P2.54mm_Vertical, F.Cu at (110.0, 180.7)
- U1: footprint RF_Module:ESP32-C3-WROOM-02 -> Custom board:ESP32-C3-WROOM-02 mod
Routing:
- net GND: vias 47 -> 56
