File: Proyecto final/Kicad/Guantes traductores/usbc.kicad_sch (KiCad schematic)
At the start: 11 parts, among them J1 USB_C_Receptacle_USB2.0_16P, U3 USBLC6-2SC6

Commit message: Posicion de componentes
Parts:
- removed R13: 5.1k, Resistor_SMD:R_0805_2012Metric_Pad1.20x1.40mm_HandSolder, symbol Device:R
- added C4: 100nF, Capacitor_SMD:C_0805_2012Metric, symbol Device:C
Connections:
- net D+: now also U3.3 (I/O2); no longer R18.1
- net D-: now also U3.1 (I/O1); no longer R17.1
- net GND: now also J1.S1 (SHIELD), C4.2
- net USB_D+: now also R18.2; no longer U3.4 (I/O2)
- net USB_D-: now also R17.2; no longer U3.6 (I/O1)
- net at C1.1, D1.1 (K), J1.A4 (VBUS)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: now also U3.5 (VBUS), C4.1
- new net: R18.1, U3.4 (I/O2)
- new net: R17.1, U3.6 (I/O1)
- no-connect marks 3 -> 2

Commit message: Avance de esquematicos
Connections:
- net R+: now reaches R18.1, U3.4 (I/O2)
- net R-: now reaches R17.1, U3.6 (I/O1)
Other:
- moved on the sheet: R17, R18
Changed lines of the file:
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@@
 	(wire
 		(pts
-			(xy 86.36 60.96) (xy 88.9 60.96)
+			(xy 86.36 60.96) (xy 95.25 60.96)
 		)
 		(stroke
@@
 	(wire
 		(pts
-			(xy 86.36 58.42) (xy 88.9 58.42)
-		)
-		(stroke
-			(width 0)
-			(type default)
+			(xy 86.36 58.42) (xy 95.25 58.42)
+		)
+		(stroke
+			(width 0)
+			(type default)
+		)
+	)
+	(label "R-"
+		(at 86.36 58.42 0)
+		(effects
+			(font
+				(size 1.27 1.27)
+			)
+			(justify left bottom)
 		)
 	)
 	(label "D-"
 		(at 58.42 58.42 0)
+		(effects
+			(font
+				(size 1.27 1.27)
+			)
+			(justify left bottom)
+		)
+	)
+	(label "R+"
+		(at 86.36 60.96 0)
 		(effects
 			(font
@@
 	(hierarchical_label "USB_D+"
 		(shape bidirectional)
-		(at 96.52 60.96 0)
+		(at 102.87 60.96 0)
 		(effects
 			(font
@@
 	(hierarchical_label "USB_D-"
 		(shape bidirectional)
-		(at 96.52 58.42 0)
+		(at 102.87 58.42 0)
 		(effects
 			(font
@@
 	(symbol
 		(lib_id "Device:R")
-		(at 92.71 60.96 90)
+		(at 99.06 60.96 90)
 		(unit 1)
 		(body_style 1)
@@
 		(dnp no)
 		(property "Reference" "R18"
-			(at 92.964 63.5 90)
+			(at 99.314 63.5 90)
 			(show_name no)
 			(do_not_autoplace no)
@@
 		)
 		(property "Value" "33"
-			(at 92.964 60.96 90)
+			(at 99.314 60.96 90)
 			(show_name no)
 			(do_not_autoplace no)
@@
 		)
 		(property "Footprint" "Resistor_SMD:R_0805_2012Metric"
-			(at 92.71 62.738 90)
+			(at 99.06 62.738 90)
 			(hide yes)
 			(show_name no)
@@
 		)
 		(property "Datasheet" ""
-			(at 92.71 60.96 0)
+			(at 99.06 60.96 0)
 			(hide yes)
 			(show_name no)
@@
 		)
 		(property "Description" "Resistor"
-			(at 92.71 60.96 0)
+			(at 99.06 60.96 0)
 			(hide yes)
 			(show_name no)
@@
 	(symbol
 		(lib_id "Device:R")
-		(at 92.71 58.42 90)
+		(at 99.06 58.42 90)
 		(unit 1)
 		(body_style 1)
@@
 		(dnp no)
 		(property "Reference" "R17"
-			(at 92.202 56.134 90)
+			(at 98.552 56.134 90)
 			(show_name no)
 			(do_not_autoplace no)
@@
 		)
 		(property "Value" "33"
-			(at 92.456 58.42 90)
+			(at 98.806 58.42 90)
 			(show_name no)
 			(do_not_autoplace no)
@@
 		)
 		(property "Footprint" "Resistor_SMD:R_0805_2012Metric"
-			(at 92.71 60.198 90)
+			(at 99.06 60.198 90)
 			(hide yes)
 			(show_name no)
@@
 		)
 		(property "Datasheet" ""
-			(at 92.71 58.42 0)
+			(at 99.06 58.42 0)
 			(hide yes)
 			(show_name no)
@@
 		)
 		(property "Description" "Resistor"
-			(at 92.71 58.42 0)
-			(hide yes)
-			(show_name no)
+			(at 99.06 58.42 0)
+			(hide yes)
+			(show_name no)
