File: Proyecto final/Kicad/Guantes traductores/sensores flex.kicad_sch (KiCad schematic)
At the start: 28 parts, among them J10 Contacto1, J11 Contacto2, J12 Contacto3, J13 Contacto4, J3 Flex1, J4 Flex2, J5 Flex3, J6 Flex4, J7 Flex5, U4 LMV324, U5 LMV324

Commit message: Posicion de componentes
Parts:
- added D10, D11, D12, D4, D5, D6, D7, D8, D9: ESD5B5.0ST1G, Diode_SMD:D_SOD-523, symbol ESD5B5.0ST1G:ESD5B5.0ST1G
Connections:
- net GND: now also D10.1, D11.1, D12.1, D4.1, D5.1, D6.1, D7.1, D8.1, D9.1
- net IO5: now also D9.2
- net IO6: now also D10.2
- net IO7: now also D12.2
- net IO8: now also D11.2
- net at C23.2, J7.2 (Pin_2), R16.2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: now also D8.2
- net at C13.2, J6.2 (Pin_2), R15.2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: now also D4.2
- net at C8.2, J3.2 (Pin_2), R22.2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: now also D7.2
- net at C12.2, J5.2 (Pin_2), R14.2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: now also D5.2
- net at C11.2, J4.2 (Pin_2), R24.2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: now also D6.2
- no-connect marks 0 -> 6
Other:
- moved on the sheet: C7, J10, J11, J12, J13, R10, R11, R12, R19, R20, R9, U5B

Commit message: Preparacion para pedido JLCPCB
Parts:
- R14, R15, R16, R22, R24: value 100k -> 250k
Changed lines of the file:
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@@
 			)
 		)
-		(property "Value" "100k"
+		(property "Value" "250k"
 			(at 173.99 47.244 90)
 			(show_name no)
@@
 			)
 		)
-		(property "Value" "100k"
+		(property "Value" "250k"
 			(at 77.47 47.244 90)
 			(show_name no)
@@
 			)
 		)
-		(property "Value" "100k"
+		(property "Value" "250k"
 			(at 138.43 47.244 90)
 			(show_name no)
@@
 			)
 		)
-		(property "Value" "100k"
+		(property "Value" "250k"
 			(at 107.95 47.244 90)
 			(show_name no)
@@
 			)
 		)
-		(property "Value" "100k"
+		(property "Value" "250k"
 			(at 46.482 48.006 90)
 			(show_name no)
