File: Proyecto final/Kicad/Guantes traductores/Esp32_C3_WROOM-02.kicad_sch (KiCad schematic)
At the start: 12 parts, among them SW1 SW_SPST, SW2 SW_SPST, U1 ESP32-C3-WROOM-02

Commit message: Ajustes vias de esp32
Parts:
- U1: footprint RF_Module:ESP32-C3-WROOM-02 -> Custom board:ESP32-C3-WROOM-02 mod
Changed lines of the file:
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@@
 			)
 		)
-		(property "Footprint" "RF_Module:ESP32-C3-WROOM-02"
+		(property "Footprint" "Custom board:ESP32-C3-WROOM-02 mod"
 			(at 149.86 64.135 0)
 			(hide yes)
